File: PTP_Karlo_Kosanovic_project1.kicad_sch (KiCad schematic)
At the start: 0 parts

Commit message: Update PTP_Karlo_Kosanovic_project1.kicad_sch
Other:
- note added: "0"
- note added: "22.10.2025."
- note added: "Karlo Kosanović"
- note added: "Projekt 1"
Changed lines of the file:
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@@
 	(generator_version "9.0")
 	(paper "A4")
+	(text "Karlo Kosanović"
+		(exclude_from_sim no)
+		(at 204.978 174.244 0)
+		(effects
+			(font
+				(size 3.81 3.81)
+			)
+		)
+	)
+	(text "22.10.2025."
+		(exclude_from_sim no)
+		(at 213.614 193.548 0)
+		(effects
+			(font
+				(size 1.27 1.27)
+			)
+		)
+	)
+	(text "0"
+		(exclude_from_sim no)
+		(at 269.24 193.548 0)
+		(effects
+			(font
+				(size 1.27 1.27)
+			)
+		)
+	)
+	(text "Projekt 1"
+		(exclude_from_sim no)
+		(at 191.77 189.738 0)
+		(effects
+			(font
+				(size 1.27 1.27)
+			)
+		)
+	)
 	(sheet_instances
 		(path "/"

Commit message: 1
Parts:
- added R1: 100R, symbol Device:R
- added R2: 100k, symbol Device:R
- added R3, R4: 2K2, symbol Device:R
Connections:
- new net: R1.2, R2.1, R3.2
- new net +3V3: R1.1
- new net GND: R2.2
- new net s: R3.1, R4.2
Other:
- note removed: "0"
- note removed: "22.10.2025."
- note removed: "Karlo Kosanović"
- note removed: "Projekt 1"
- company: (none) -> TVZ
- title: (none) -> Labaratorijske vjezbe

Commit message: vjezba 2
Parts:
- added C1: 220u, symbol Device:C_Polarized
- added C2: 22u, symbol Device:C_Polarized
- added C3: 10m, symbol Device:C_Polarized
- added C4: 100n, symbol Device:C
- added C5: 1u, symbol Device:C
- added D1: 11DQ06, symbol Device:D_Schottky
- added D2, D3, D4, D5: LED, symbol Device:LED
- added J1: Screw_Terminal_01x02, symbol Connector:Screw_Terminal_01x02
- added L1: 330u, symbol Device:L
- added R5, R6, R7, R8: 4k7, symbol Device:R
- added SW1: SW_Push, symbol Switch:SW_Push
- added SW2: SW_Wuerth_450301014042, Button_Switch_THT:SW_Slide-03_Wuerth-WS-SLTV_10x2.5x6.4_P2.54mm, symbol Switch:SW_Wuerth_450301014042
- added U1: LM2574N-5, Package_DIP:DIP-8_W7.62mm, symbol Regulator_Switching:LM2574N-5
- added U2: NE555P, Package_DIP:DIP-8_W7.62mm, symbol Timer:NE555P
- R1: value 100R -> 47k
- R2: value 100k -> 47k
- R3: value 2K2 -> 10k
- R4: value 2K2 -> 2k
Connections:
- net GND: now also C1.2, C2.2, C3.2, C4.2, C5.1, D1.2 (A), J1.1 (Pin_1), R5.2, R6.2, R7.2, R8.2, SW1.1, U1.2 (SGND), U1.3 (~{ON}/OFF), U1.4 (PGND), U2.1 (GND); no longer R2.2
- net at R4.1: now also SW1.2
- net at R1.2, R2.1: now also U2.7 (DIS); no longer R3.2
- net +3V3 renamed +5V
- net +5V: now also R3.1, C1.1, C4.1, L1.2, U1.1 (FB), U2.4 (R), U2.8 (VCC)
- net s: no longer names the net of R4.2
- net s: now also C5.2, SW2.3 (A); no longer R3.1
- new net: D3.1 (K), R6.1
- new net: C3.1, R2.2, U2.2 (TR), U2.6 (THR)
- new net: D4.1 (K), R7.1
- new net: D5.1 (K), R8.1
- new net: D2.1 (K), R5.1
- new net: D1.1 (K), L1.1, U1.7 (OUT)
- new net 555: SW2.2 (C), U2.3 (Q)
- new net Q0: D2.2 (A)
- new net Q1: D3.2 (A)
- new net Q2: D4.2 (A)
- new net Q3: D5.2 (A)
- new net VDD: C2.1, J1.2 (Pin_2), U1.5 (VIN)
- new net clock: R3.2, SW2.1 (B)
- no-connect marks 0 -> 1

Commit message: a
a
Parts:
- C1: value 220u -> C_Polarized
- C2: value 22u -> C_Polarized
- C3: value 10m -> C_Polarized
- C4: value 100n -> C
- C5: value 1u -> C
- D1: value 11DQ06 -> D_Schottky
- L1: value 330u -> L
- R1, R2: value 47k -> R
- R3: value 10k -> R
- R4: value 2k -> R
- R5, R6, R7, R8: value 4k7 -> R
Changed lines of the file:
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@@
 			)
 		)
-		(property "Value" "4k7"
+		(property "Value" "R"
 			(at 191.77 30.48 90)
 			(effects
@@
 		(on_board yes)
 		(dnp no)
-		(property "Reference" "#PWR04"
+		(property "Reference" "#PWR4"
 			(at 60.96 50.8 0)
 			(effects
@@
 		)
 		(property "Value" "GND"
-			(at 60.96 52.07 0)
+			(at 60.96 48.26 0)
 			(effects
 				(font
@@
 			(project ""
 				(path "/e13bcad6-39aa-4cc7-a96a-2fdaddc66971"
-					(reference "#PWR04")
+					(reference "#PWR4")
 					(unit 1)
 				)
@@
 			)
 		)
-		(property "Value" "22u"
+		(property "Value" "C_Polarized"
 			(at 39.37 33.4009 0)
 			(effects
@@
 		(dnp no)
 		(fields_autoplaced yes)
-		(property "Reference" "#PWR03"
+		(property "Reference" "#PWR3"
 			(at 35.56 24.13 0)
 			(effects
@@
 			(project ""
 				(path "/e13bcad6-39aa-4cc7-a96a-2fdaddc66971"
-					(reference "#PWR03")
+					(reference "#PWR3")
 					(unit 1)
 				)
@@
 		(dnp no)
 		(fields_autoplaced yes)
-		(property "Reference" "#PWR08"
+		(property "Reference" "#PWR8"
 			(at 35.56 101.6 0)
 			(effects
@@
 			(project ""
 				(path "/e13bcad6-39aa-4cc7-a96a-2fdaddc66971"
-					(reference "#PWR08")
+					(reference "#PWR8")
 					(unit 1)
 				)
@@
 			)
 		)
-		(property "Value" "47k"
+		(property "Value" "R"
 			(at 20.32 101.5999 0)
 			(effects
@@
 		(dnp no)
 		(fields_autoplaced yes)
-		(property "Reference" "#PWR02"
+		(property "Reference" "#PWR2"
 			(at 29.21 44.45 0)
 			(effects
@@
 			(project ""
 				(path "/e13bcad6-39aa-4cc7-a96a-2fdaddc66971"
-					(reference "#PWR02")
+					(reference "#PWR2")
 					(unit 1)
 				)
@@
 			)
 		)
-		(property "Value" "4k7"
+		(property "Value" "R"
 			(at 191.77 53.34 90)
 			(effects
@@
 			)
 		)
-		(property "Value" "4k7"
+		(property "Value" "R"
 			(at 191.77 19.05 90)
 			(effects
@@
 		(dnp no)
 		(fields_autoplaced yes)
-		(property "Reference" "#PWR07"
+		(property "Reference" "#PWR7"
 			(at 52.07 83.82 0)
 			(effects
@@
 			(project ""
 				(path "/e13bcad6-39aa-4cc7-a96a-2fdaddc66971"
-					(reference "#PWR07")
+					(reference "#PWR7")
 					(unit 1)
 				)
@@
 			)
 		)
-		(property "Value" "10k"
+		(property "Value" "R"
 			(at 68.58 59.6899 0)
 			(effects
@@
 		(dnp no)
 		(fields_autoplaced yes)
-		(property "Reference" "#PWR010"
+		(property "Reference" "#PWR10"
 			(at 66.04 57.15 0)
 			(effects
@@
 			(project "PTP_Karlo_Kosanovic_project1"
 				(path "/e13bcad6-39aa-4cc7-a96a-2fdaddc66971"
-					(reference "#PWR010")
+					(reference "#PWR10")
 					(unit 1)
 				)
@@
 			)
 		)
-		(property "Value" "47k"
+		(property "Value" "R"
 			(at 20.32 92.7099 0)
 			(effects
@@
 		(dnp no)
 		(fields_autoplaced yes)
-		(property "Reference" "#PWR09"
+		(property "Reference" "#PWR9"
 			(at 19.05 69.85 0)
 			(effects
@@
 			(project ""
 				(path "/e13bcad6-39aa-4cc7-a96a-2fdaddc66971"
-					(reference "#PWR09")
+					(reference "#PWR9")
 					(unit 1)
 				)
@@
 			)
 		)
-		(property "Value" "330u"
+		(property "Value" "L"
 			(at 78.74 30.48 90)
 			(effects
@@
 			)
 		)
-		(property "Value" "10m"
+		(property "Value" "C_Polarized"
 			(at 21.59 118.4909 0)
 			(effects
@@
 			)
 		)
-		(property "Value" "2k"
+		(property "Value" "R"
 			(at 39.37 57.15 90)
 			(effects
@@
 		(dnp no)
 		(fields_autoplaced yes)
-		(property "Reference" "#PWR01"
+		(property "Reference" "#PWR1"
 			(at 29.21 22.86 0)
 			(effects
@@
 			(project ""
 				(path "/e13bcad6-39aa-4cc7-a96a-2fdaddc66971"
-					(reference "#PWR01")
+					(reference "#PWR1")
 					(unit 1)
 				)
@@
 			)
 		)
-		(property "Value" "4k7"
+		(property "Value" "R"
 			(at 191.77 41.91 90)
 			(effects
@@
 			)
 		)
-		(property "Value" "100n"
+		(property "Value" "C"
 			(at 39.37 88.8999 0)
 			(effects
@@
 			)
 		)
-		(property "Value" "1u"
+		(property "Value" "C"
 			(at 34.29 46.99 90)
 			(effects
@@
 		(dnp no)
 		(fields_autoplaced yes)
-		(property "Reference" "#PWR06"
+		(property "Reference" "#PWR6"
 			(at 17.78 130.81 0)
 			(effects
@@
 			(project ""
 				(path "/e13bcad6-39aa-4cc7-a96a-2fdaddc66971"
-					(reference "#PWR06")
+					(reference "#PWR6")
 					(unit 1)
 				)
@@
 		(dnp no)
 		(fields_autoplaced yes)
-		(property "Reference" "#PWR011"
+		(property "Reference" "#PWR11"
 			(at 199.39 68.58 0)
 			(effects
@@
 			(project ""
 				(path "/e13bcad6-39aa-4cc7-a96a-2fdaddc66971"
-					(reference "#PWR011")
+					(reference "#PWR11")
 					(unit 1)
 				)
@@
 		(dnp no)
 		(property "Reference" "SW2"
-			(at 52.07 72.39 0)
+			(at 52.07 58.42 0)
 			(effects
 				(font
@@
 		)
 		(property "Value" "SW_Wuerth_450301014042"
-			(at 52.07 69.85 0)
+			(at 52.07 68.58 0)
 			(effects
 				(font
@@
 			)
 		)
-		(property "Value" "11DQ06"
+		(property "Value" "D_Schottky"
 			(at 74.93 39.0524 90)
 			(effects
@@
 		(dnp no)
 		(fields_autoplaced yes)
-		(property "Reference" "#PWR05"
+		(property "Reference" "#PWR5"
 			(at 85.09 25.4 0)
 			(effects
@@
 			(project ""
 				(path "/e13bcad6-39aa-4cc7-a96a-2fdaddc66971"
-					(reference "#PWR05")
+					(reference "#PWR5")
 					(unit 1)
 				)
@@
 			)
 		)
-		(property "Value" "220u"
+		(property "Value" "C_Polarized"
 			(at 88.9 38.4809 0)
 			(effects

Commit message: cila schema
Parts:
- added H1, H2, H3, H4: MountingHole, symbol Mechanical:MountingHole
- added R10, R11, R12, R15, R9: 10k, symbol Device:R
- added R14, R16, R17, R18, R5, R6, R8: 2k, symbol Device:R
- added U3: 74LVC1G11, symbol 74xGxx:74LVC1G11
- added U4, U5: 4027, symbol 4xxx:4027
- added U5: FYS-3911BUHR-21, Display_7Segment:HDSP-7401, symbol Display_Character:HDSP-7401
- C3: value C_Polarized -> 10u
- C4: value C -> 100n
- C5: value C -> 1u
- R1, R2: value R -> 47k
- R3: value R -> 10k
- R4: value R -> 2k
- R5, R6, R7, R8: value R -> 4k7
Connections:
- net +5V: now also R10.1, R11.1, R12.1, R15.1, R9.1, U3.5 (VCC), U4.16 (VCC), U4.16 (VDD), U5.1 (CA), U5.16 (VDD), U5.6 (CA)
- net GND: now also U3.2 (GND), U4.7 (S), U4.8 (GND), U4.8 (VSS), U4.9 (S), U5.7 (S), U5.8 (VSS), U5.9 (S)
- net Q0: now also U4.1 (Q), U4.13 (C), U4.7 (A)
- net Q1: now also U3.6, U4.1 (B), U4.15 (Q), U5.3 (C)
- net Q2: now also U4.2 (C), U5.1 (Q), U5.13 (C)
- net Q3: now also U3.1, U4.6 (D), U5.15 (Q)
- net clock renamed Clock
- net Clock: now also U3.3, U4.3 (C)
- new net: R5.2, U5.10 (A)
- new net: R17.2, U5.2 (F)
- new net: R18.2, U5.3 (G)
- new net: R16.2, U5.4 (E)
- new net: R14.2, U5.5 (D)
- new net: R8.2, U5.8 (C)
- new net: R6.2, U5.9 (B)
- new net: R6.1, U4.12 (b)
- new net: R10.2, U4.10 (J), U4.11 (K)
- new net: R14.1, U4.10 (d)
- new net: R9.2, U4.5 (K), U4.6 (J)
- new net: R8.1, U4.11 (c)
- new net: R5.1, U4.13 (a)
- new net: R18.1, U4.14 (g)
- new net: R17.1, U4.15 (f)
- new net: R15.2, U4.5 (RBI)
- new net: R16.1, U4.9 (e)
- new net: R11.2, U5.5 (K), U5.6 (J)
- new net: R12.2, U5.10 (J), U5.11 (K)
- new net Reset: U3.4
- no-connect marks 1 -> 6
Other:
- note added: "555 timer"
- note added: "JK bistabili"
- note added: "LED diode"
- note added: "Montažne rupe"
- note added: "Napajanje"
- note added: "Napajanje bistabila"
- note added: "Reset brojača"
- note added: "Tipkalo i ulaz radnog takta"
- moved on the sheet: C1, C2, C3, C4, C5, D1, D2, D3, D4, D5, J1, L1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

Commit message: schema gotovija nego prije
Parts:
- renumbered R5 to R1, R4 to R13, R1 to R19, R6 to R2, R2 to R20, R7 to R3, R8 to R4, R3 to R7, U4 to U2, U5 to U3, U3 to U6, U2 to U7
Connections:
- net Reset: now also U2.12 (R), U2.4 (R), U3.12 (R), U3.4 (R)
- net at U4.3 (LT): now also R15.2, U4.4 (BI), U4.5 (RBI)
Other:
- moved on the sheet: J1
