File: PTP_Karlo_Kosanovic_project1.kicad_sch (KiCad schematic)
At the start: 45 parts, among them J1 Screw_Terminal_01x02, SW1 SW_Push, SW2 SW_Wuerth_450301014042, U1 LM2574N-5, U2 4027, U3 4027, U4 74LS47, U5 FYS-3911BUHR-21, U6 74LVC1G11, U7 NE555P

Commit message: a
a
Parts:
- D1: value D_Schottky -> LED
- D4: footprint LED_THT:LED_D5.0mm -> Diode_THT:D_DO-41_SOD81_P12.70mm_Horizontal
Changed lines of the file:
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@@
 			)
 		)
-		(property "Footprint" "LED_THT:LED_D5.0mm"
+		(property "Footprint" "Diode_THT:D_DO-41_SOD81_P12.70mm_Horizontal"
 			(at 242.57 45.72 0)
 			(effects
@@
 			)
 		)
-		(property "Value" "D_Schottky"
+		(property "Value" "LED"
 			(at 88.9 47.9424 90)
 			(effects
