File: PTP_Karlo_Kosanovic_project1.kicad_pcb (KiCad board)
At the start: 2 copper layers, 45 parts, among them J1 Screw_Terminal_01x02, SW1 SW_Push, SW2 SW_Wuerth_450301014042, U1 LM2574N-5, U2 4027, U3 4027, U4 74LS47, U5 FYS-3911BUHR-21, U6 74LVC1G11, U7 NE555P

Commit message: a
a
Parts:
- D1: value D_Schottky -> LED
- moved H4 251.9 mm to (204.5, 147.5)
- moved H3 240.7 mm to (204.5, 49.5)
- moved H2 163.2 mm to (93.0, 147.5)
- moved H1 129.8 mm to (93.0, 49.5)
- moved D2 127.0 mm to (170.8, 75.8), turned to -90 degrees
- moved R1 125.3 mm to (171.1, 57.1), turned to -90 degrees
- moved R2 114.5 mm to (164.1, 56.9), turned to -90 degrees
- moved D4 113.5 mm to (148.9, 70.0)
- moved D3 112.7 mm to (163.4, 75.8), turned to -90 degrees
- moved U6 106.2 mm to (161.1, 113.8)
- moved R3 103.4 mm to (156.6, 56.9), turned to -90 degrees
- moved D5 98.7 mm to (155.9, 76.0), turned to -90 degrees
- moved L1 96.8 mm to (129.4, 81.8), turned to 90 degrees
- moved R4 92.4 mm to (149.1, 56.9), turned to -90 degrees
- moved J1 88.9 mm to (106.3, 82.8)
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