File: projekt/projekt.kicad_sch (KiCad schematic)
At the start: 45 parts, among them J1 Screw_Terminal_01x02, SW1 SW_Push, SW2 SW_Wuerth_450301014042, U1 LM2574N-5, U2 4027, U3 4027, U4 74LS47, U5 FYS-3911BUHR-21, U6 74LVC1G11, U7 NE555P

Commit message: a
Parts:
- C1, C2: footprint Capacitor_THT:CP_Radial_D5.0mm_P2.00mm -> (none)
- C3, C4, C5: footprint Capacitor_SMD:C_1206_3216Metric_Pad1.33x1.80mm_HandSolder -> (none)
- D1, D2, D3, D4, D5: footprint LED_THT:LED_D5.0mm -> (none)
- H1, H2, H3, H4: footprint MountingHole:MountingHole_5.5mm -> (none)
- J1: footprint TerminalBlock_MetzConnect:TerminalBlock_MetzConnect_Type011_RT05502HBLC_1x02_P5.00mm_Horizontal -> (none)
- L1: footprint Inductor_THT:L_Radial_D7.2mm_P3.00mm_Murata_1700 -> (none)
- R1, R2, R3, R4: footprint Resistor_THT:R_Axial_DIN0207_L6.3mm_D2.5mm_P10.16mm_Horizontal -> (none)
- R10, R11, R12, R13, R14, R15, R16, R17, R18, R19, R20, R5, R6, R7, R8, R9: footprint Resistor_SMD:R_1206_3216Metric_Pad1.30x1.75mm_HandSolder -> (none)
- SW1: footprint Button_Switch_THT:SW_PUSH_6mm_H4.3mm -> (none)
- SW2: footprint Button_Switch_THT:SW_Slide_SPDT_Straight_CK_OS102011MS2Q -> Button_Switch_THT:SW_Slide-03_Wuerth-WS-SLTV_10x2.5x6.4_P2.54mm
- U1: footprint Package_DIP:DIP-8_W7.62mm_Socket_LongPads -> Package_DIP:DIP-8_W7.62mm
- U2, U3, U4: footprint Package_DIP:DIP-16_W7.62mm_Socket_LongPads -> (none)
- U6: footprint Package_TO_SOT_SMD:SOT-23-6 -> (none)

Commit message: a
a
Parts:
- C1, C2: footprint (none) -> Capacitor_THT:CP_Radial_D5.0mm_P2.00mm
- C3, C4, C5: footprint (none) -> Capacitor_SMD:C_1206_3216Metric_Pad1.33x1.80mm_HandSolder
- D1: value D_Schottky -> LED; footprint (none) -> LED_THT:LED_D5.0mm
- D2, D3, D5: footprint (none) -> LED_THT:LED_D5.0mm
- D4: footprint (none) -> Diode_THT:D_DO-41_SOD81_P12.70mm_Horizontal
- H1, H2, H3, H4: footprint (none) -> MountingHole:MountingHole_5.5mm
- J1: footprint (none) -> TerminalBlock_MetzConnect:TerminalBlock_MetzConnect_Type011_RT05502HBLC_1x02_P5.00mm_Horizontal
- L1: footprint (none) -> Inductor_THT:L_Radial_D7.2mm_P3.00mm_Murata_1700
- R1, R2, R3, R4: footprint (none) -> Resistor_THT:R_Axial_DIN0207_L6.3mm_D2.5mm_P10.16mm_Horizontal
- R10, R11, R12, R13, R14, R15, R16, R17, R18, R19, R20, R5, R6, R7, R8, R9: footprint (none) -> Resistor_SMD:R_1206_3216Metric_Pad1.30x1.75mm_HandSolder
- SW1: footprint (none) -> Button_Switch_THT:SW_PUSH_6mm_H4.3mm
- SW2: footprint Button_Switch_THT:SW_Slide-03_Wuerth-WS-SLTV_10x2.5x6.4_P2.54mm -> Button_Switch_THT:SW_Slide_SPDT_Straight_CK_OS102011MS2Q
- U1: footprint Package_DIP:DIP-8_W7.62mm -> Package_DIP:DIP-8_W7.62mm_Socket_LongPads
- U2, U3, U4: footprint (none) -> Package_DIP:DIP-16_W7.62mm_Socket_LongPads
- U6: footprint (none) -> Package_TO_SOT_SMD:SOT-23-6
