File: projekt/projekt.kicad_pcb (KiCad board)
At the start: 2 copper layers, 45 parts, among them J1 Screw_Terminal_01x02, SW1 SW_Push, SW2 SW_Wuerth_450301014042, U1 LM2574N-5, U2 4027, U3 4027, U4 74LS47, U5 FYS-3911BUHR-21, U6 74LVC1G11, U7 NE555P

Commit message: a
Parts:
- moved R15 25.8 mm to (204.5, 96.0), turned to 90 degrees
- moved R1 24.3 mm to (148.9, 66.9), turned to 90 degrees
- moved R4 24.0 mm to (170.9, 67.1), turned to 90 degrees
- moved D2 20.9 mm to (150.0, 76.0)
- moved D4 15.7 mm to (164.5, 71.0)
- moved D5 15.6 mm to (171.5, 76.0)
- moved R2 13.1 mm to (155.9, 67.1), turned to 90 degrees
- moved R3 12.2 mm to (163.4, 67.1), turned to 90 degrees
- moved U5 9.52 mm to (194.5, 90.9)
- moved R10 7.54 mm to (108.0, 104.5)
- moved R11 7.54 mm to (108.0, 107.0)
- moved R12 7.54 mm to (108.0, 109.5)
- moved R9 7.54 mm to (108.0, 102.0)
- moved R18 7.04 mm to (184.5, 94.0)
- moved R8 6.28 mm to (184.6, 101.5)
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Routing:
- net +5V: track 0.00 -> 222.8 mm
- net GND: track 0.00 -> 194.5 mm, vias 0 -> 2
- net Q1: track 0.00 -> 51.3 mm
- net Net-(U7-THR): track 0.00 -> 45.0 mm
- net Net-(U2A-J): track 0.00 -> 42.6 mm
- net Clock: track 0.00 -> 26.1 mm
- net Q0: track 0.00 -> 22.9 mm
- net Reset: track 0.00 -> 22.9 mm
- net 555: track 0.00 -> 20.6 mm
- net VDD: track 0.00 -> 18.2 mm
- net Net-(U5-D): track 0.00 -> 17.3 mm
- net Q3: track 0.00 -> 12.2 mm
- net Net-(U5-E): track 0.00 -> 11.7 mm
- net Net-(R13-Pad1): track 0.00 -> 11.6 mm
- net (no net): track 0.00 -> 10.9 mm
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